File: pcb_files/school_meteo.kicad_sch (KiCad schematic)
At the start: 49 parts, among them J1 4P4C, J2 4P4C, J3 4P4C, J4 8P8C_MAG_POE_LED, U1 ESP32, U2 WIZNET_W5500, U4 LM2592HVSX-3.3, Y1 25MHz

Commit message: Updating schematic
Updating schematic
Parts:
- removed C10, C11, C7: 0.1uF, symbol Device:C
- removed C13, C8: 10uF, symbol Device:C
- removed C18: 6.8nF, symbol Device:C
- removed C4, C6: C, symbol Device:C
- removed D1: D_Schottky, Package_TO_SOT_SMD:TO-252-3_TabPin4, symbol Device:D_Schottky
- removed J1, J2, J3: 4P4C, symbol Connector:4P4C
- removed R1: 1k, symbol Device:R
- removed R11, R9: 10K, symbol Device:R
- removed R3: 10k, symbol Device:R
- removed U1: ESP32, School_meteo:ESP-WROOM-32, symbol ESP32:ESP32
- added C10, C4, C6: 10uF, Capacitor_THT:CP_Radial_D5.0mm_P2.00mm, symbol Device:C_Polarized
- added C2: 18pF, Capacitor_THT:C_Rect_L4.6mm_W3.0mm_P2.50mm_MKS02_FKP02, symbol Device:C
- added C5, C9: 0.1uF, Capacitor_THT:C_Rect_L4.6mm_W3.0mm_P2.50mm_MKS02_FKP02, symbol Device:C
- added D1: MBRD20150CT, Package_TO_SOT_SMD:TO-252-3_TabPin4, symbol School_meteo:MBRD20150CT
- added H1, H2, H3, H4: MountingHole, MountingHole:MountingHole_3.2mm_M3_DIN965_Pad, symbol Mechanical:MountingHole
- added J1, J2, J3: 4P4C, School_meteo:4P4C, symbol School_meteo:4P4C
- added R12: 1k, Resistor_THT:R_Axial_DIN0204_L3.6mm_D1.6mm_P5.08mm_Horizontal, symbol Device:R
- added R4: 470, Resistor_THT:R_Axial_DIN0204_L3.6mm_D1.6mm_P5.08mm_Horizontal, symbol Device:R
- added R5, R6: 10K, Resistor_THT:R_Axial_DIN0204_L3.6mm_D1.6mm_P5.08mm_Horizontal, symbol Device:R
- added U1: ESP-WROOM-32, School_meteo:ESP-WROOM-32, symbol School_meteo:ESP-WROOM-32
- C1: renamed from C3; value C -> 18pF; footprint (none) -> Capacitor_THT:C_Rect_L4.6mm_W3.0mm_P2.50mm_MKS02_FKP02; Name (none) -> K180J15C0GF53L2
- C11: renamed from C1; footprint (none) -> Capacitor_THT:C_Rect_L4.6mm_W3.8mm_P2.50mm_MKS02_FKP02; Name (none) -> FG18X7R1E105KRT00
- C12: value 0.1uF -> 10nF; footprint (none) -> Capacitor_THT:C_Rect_L4.6mm_W3.0mm_P2.50mm_MKS02_FKP02; Name (none) -> K103Z15Y5VF5TL2
- C13: renamed from C15; footprint Capacitor_THT:CP_Radial_D5.0mm_P2.00mm -> Capacitor_THT:CP_Radial_D6.3mm_P2.50mm; Name ESK226M025AC3AA -> 32SEPF22M+TSS
- C14: footprint (none) -> Capacitor_THT:C_Rect_L4.6mm_W3.0mm_P2.50mm_MKS02_FKP02; Name (none) -> K103Z15Y5VF5TL2
- C15: renamed from C17; footprint (none) -> Capacitor_THT:C_Rect_L4.6mm_W3.0mm_P2.50mm_MKS02_FKP02; Name (none) -> FG18X7R1H682KNT00
- C16: value 10nF -> 6.8nF; footprint (none) -> Capacitor_THT:C_Rect_L4.6mm_W3.0mm_P2.50mm_MKS02_FKP02; Name (none) -> FG18X7R1H682KNT00
- C17: renamed from C19; footprint Capacitor_THT:C_Disc_D5.0mm_W2.5mm_P2.50mm -> Capacitor_THT:C_Rect_L4.6mm_W3.0mm_P2.50mm_MKS02_FKP02
- C3: renamed from C5; value C -> 10nF; footprint (none) -> Capacitor_THT:C_Rect_L4.6mm_W3.0mm_P2.50mm_MKS02_FKP02; Name (none) -> K103Z15Y5VF5TL2
- C7: renamed from C2; footprint (none) -> Capacitor_THT:C_Rect_L4.6mm_W3.8mm_P2.50mm_MKS02_FKP02; Name (none) -> FG18X7R1E105KRT00
- C8: renamed from C9; footprint (none) -> Capacitor_THT:C_Rect_L4.6mm_W3.0mm_P2.50mm_MKS02_FKP02; Name (none) -> K104M15X7RF53H5
- FB1, FB2: footprint (none) -> School_meteo:Ferrite_bead_0805; Name (none) -> BLM21PG121SH1D
- J4: renamed from J?; value Push-In_terminal_block -> Terminal_block; footprint TerminalBlock:TerminalBlock_bornier-2_P5.08mm -> School_meteo:Phoenix_LPT_2,5_2-5,0; Name (none) -> LPT 2,5/ 2-5,0
- J5: renamed from J4; footprint (none) -> School_meteo:TE_Connectivity_PoE
- R1: renamed from R4; footprint (none) -> Resistor_THT:R_Axial_DIN0204_L3.6mm_D1.6mm_P5.08mm_Horizontal; Name (none) -> CFS1/4CT52R105J
- R10, R8: footprint (none) -> Resistor_THT:R_Axial_DIN0204_L3.6mm_D1.6mm_P5.08mm_Horizontal; Name (none) -> CFS1/4CT52R103J
- R11: renamed from R12; footprint (none) -> Resistor_THT:R_Axial_DIN0207_L6.3mm_D2.5mm_P7.62mm_Horizontal; Name (none) -> MF1/4DCT52R1242F
- R13, R14, R15, R16: footprint (none) -> Resistor_THT:R_Axial_DIN0207_L6.3mm_D2.5mm_P7.62mm_Horizontal; Name (none) -> MF1/4DCT52R49R9F
- R17: footprint (none) -> Resistor_THT:R_Axial_DIN0207_L6.3mm_D2.5mm_P7.62mm_Horizontal; Name (none) -> MF1/4DCT52R10R0F
- R2: renamed from R5; footprint (none) -> Resistor_THT:R_Axial_DIN0204_L3.6mm_D1.6mm_P5.08mm_Horizontal; Name (none) -> CFS1/4CT52R103J
- R3: renamed from R6; footprint (none) -> Resistor_THT:R_Axial_DIN0204_L3.6mm_D1.6mm_P5.08mm_Horizontal; Name (none) -> CFS1/4CT52R471J
- R7: value 470 -> 10K; footprint (none) -> Resistor_THT:R_Axial_DIN0204_L3.6mm_D1.6mm_P5.08mm_Horizontal; Name (none) -> CFS1/4CT52R103J
- R9: renamed from R2; footprint (none) -> Resistor_THT:R_Axial_DIN0204_L3.6mm_D1.6mm_P5.08mm_Horizontal; Name (none) -> CFS1/4CT52R102J
- Y1: footprint (none) -> Crystal:Crystal_HC49-U_Vertical; Name (none) -> ECS-250-18-4X-CKM
- renumbered U4 to U3
Connections:
- net +3V3: now also R7.2, C4.1, J1.1, R12.1, R5.2, R6.2, U1.1 (+3.3)
- net GND: now also C2.2, C4.2, D1.1 (A), J1.4, J2.1, J2.2, J3.2, U1.38 (GND)
- net GNDA: now also C14.2, C10.2, C5.2, C6.2, C9.2; no longer C14.1, C16.1
- net GREENLED: now also R4.1; no longer R7.1
- net MISO: now also U1.31 (GPIO19)
- net MOSI: now also U1.37 (GPIO23)
- net RX-: now also C16.1
- net Rain: now also J3.3, R12.2, U1.9 (GPIO25)
- net SCK: now also U1.30 (GPIO18)
- net SCL: now also J1.3, U1.36 (GPIO22)
- net SCS: now also U1.29 (GPIO5)
- net SDA: now also J1.2, U1.33 (GPIO21)
- net VDDA: now also C8.1, U2.11 (AVDD), U2.4 (AVDD), U2.8 (AVDD), C10.1, C9.1
- net Wind dir: now also R10.1, J2.4, U1.6 (GPIO35)
- net Wind speed: now also J2.3, U1.12 (GPIO14)
- net at L1.1, U3.2 (OUT): now also D1.4 (K)
- net at R1.2, U2.30 (XI/CLKIN), Y1.2: now also C2.1
- net at U2.43 (PMODE2): now also R6.1
- net at U2.44 (PMODE1): now also R7.1; no longer R10.1
- net at U2.22 (1V20): now also C5.1
- net at J5.6 (RX-): now also C16.2
- net at U2.20 (TOCAP): now also C6.1
- net at U2.25 (LINKLED): now also R4.2; no longer R7.2
- net at U2.37 (RSTn): now also R5.1; no longer R8.1
- net at U2.45 (PMODE0): now also R8.1
- net at J5.7 (RTC), R14.2, R16.2: now also C14.1; no longer C16.2
- net at J5.4 (TCT), R17.2: now also C12.1; no longer C14.2
- no-connect marks 15 -> 45
Other:
- note added: "Mounting holes"
- moved on the sheet: C11, J4
